File: Kartrack_Main_Board/ALIM .kicad_sch (KiCad schematic)
At the start: 23 parts, among them IC1 MIC3172YM, J4 Conn_01x02_Socket, U1 MIC5219-3.3YM5, U4 BQ21040DBV

Commit message: add filtering button
Parts:
- U1: MPN (none) -> MIC5219-3.3YM5-TR
Changed lines of the file:
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@@
+			)
+		)
+		(property "MPN" "MIC5219-3.3YM5-TR"
+			(at 60.96 82.55 0)
+			(effects
+				(font
+					(size 1.27 1.27)
+				)
+				(hide yes)
 			)
 		)
