File: Kartrack_Main_Board/ALIM .kicad_sch (KiCad schematic)
At the start: 0 parts

Commit message: schematic GPS
Parts:
- added C1: 2.2uF, symbol Device:C_Small
- added C2: 470pF, symbol Device:C_Small
- added U1: MIC5219-3.3YM5, Package_TO_SOT_SMD:SOT-23-5, symbol Regulator_Linear:MIC5219-3.3YM5
Connections:
- new net: C2.1, U1.4 (BP)
- new net +3.3V: C1.1, U1.5 (OUT)
- new net +5V: U1.1 (IN), U1.3 (EN)
- new net GND: C1.2, C2.2, U1.2 (GND)

Commit message: buck schematic
Parts:
- added C8: 22uF, symbol Device:C
- added C9: 15pf, symbol Device:C_Small
- added D2: LED, symbol Device:LED
- added D3, D4: D, symbol Device:D
- added D5: 5V, symbol Device:D_Zener
- added IC1: MIC3172YM, SOIC127P599X173-8N, symbol MIC3172YM:MIC3172YM
- added L2: L, symbol Device:L
- added R10, R12, R13: 1k, symbol Device:R_Small
- added R11: 0, symbol Device:R_Small
- added R14: RISET, symbol Device:R_Small
- added R9: 10k, symbol Device:R_Small
- added U4: BQ21040DBV, Package_TO_SOT_SMD:SOT-23-6, symbol Battery_Management:BQ21040DBV
Connections:
- net +5V: now also C8.1, C9.1, D4.1 (K), D5.1 (K), R12.1, U4.6 (VIN)
- net GND: now also C8.2, D5.2 (A), IC1.1 (S_GND), IC1.6 (P_GND_2), IC1.8 (P_GND_1), R13.2, R14.2, U4.5 (GND)
- new net: R14.1, U4.4 (ISET)
- new net: D4.2 (A), IC1.7 (VSW), L2.2
- new net: D3.1 (K), IC1.5 (VIN), L2.1, R11.1
- new net: D2.1 (K), U4.3 (~{CHG})
- new net: D2.2 (A), R10.2
- new net: IC1.4 (~{SYNC}/EN), R11.2
- new net: C9.2, IC1.3 (FB), R12.2, R13.1
- new net +BATT: D3.2 (A), R10.1, R9.1, U4.2 (OUT)
- new net -BATT: R9.2, U4.1 (TS)

Commit message: buck verif
Parts:
- removed D4: D, symbol Device:D
- added C10: 1uF, symbol Device:C_Small
- added C7: C, symbol Device:C
- added D4: 1N5822, Diode_THT:D_DO-201AD_P15.24mm_Horizontal, symbol Diode:1N5822
- added J4: Conn_01x02_Socket, symbol Connector:Conn_01x02_Socket
- added R15: 0, symbol Device:R_Small
- added R16: 1k, symbol Device:R_Small
- C8: value 22uF -> 470uF
- L2: value L -> 120uH
- R12: value 1k -> 3,74k
- R13: value 1k -> 1,24k
Connections:
- net +5V: now also D4.1 (K)
- net +BATT: now also J4.1 (Pin_1)
- net -BATT: now also J4.2 (Pin_2)
- net GND: now also C10.2, C7.2, R15.2
- net at IC1.7 (VSW), L2.2: now also D4.2 (A)
- net at D3.1 (K), IC1.5 (VIN), L2.1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: now also C7.1
- net at IC1.4 (~{SYNC}/EN), R11.2: now also R15.1
- net at IC1.2 (COMP): now also R16.1
- new net: C10.1, R16.2
Other:
- note added: "FeedBack of 1.240V"
- moved on the sheet: D3

Commit message: update
Parts:
- removed D3: D, symbol Device:D
- removed D5: 5V, symbol Device:D_Zener
- added D3: BZX84W, Package_TO_SOT_SMD:SOT-23, symbol Diode:BZX84Cxx
- C1, C10, C2, C9: footprint (none) -> Capacitor_SMD:C_0603_1608Metric
- C7: value C -> 10uF; footprint (none) -> Capacitor_SMD:C_0603_1608Metric
- C8: value 470uF -> 47uF; footprint (none) -> Capacitor_SMD:C_0603_1608Metric
- L2: footprint (none) -> Inductor_SMD:L_12x12mm_H8mm
- R10, R11, R12, R13, R14, R15, R16, R9: footprint (none) -> Resistor_SMD:R_0201_0603Metri
Connections:
- net +5V: now also D3.3 (K)
- net +BATT: now also C7.1, IC1.5 (VIN), L2.1, R11.1
- net GND: now also D3.1 (A)
Changed lines of the file:
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@@
 	(text "FeedBack of 1.240V \n"
 		(exclude_from_sim no)
-		(at 230.124 53.086 0)
+		(at 235.712 59.944 0)
 		(effects
 			(font
@@
 	(wire
 		(pts
-			(xy 167.64 71.12) (xy 168.91 71.12)
-		)
-		(stroke
-			(width 0)
-			(type default)
-		)
-	)
-	(wire
-		(pts
 			(xy 223.52 71.12) (xy 228.6 71.12)
 		)
@@
 	(wire
 		(pts
-			(xy 156.21 71.12) (xy 160.02 71.12)
+			(xy 156.21 71.12) (xy 168.91 71.12)
 		)
 		(stroke
@@
 			)
 		)
-		(property "Footprint" ""
+		(property "Footprint" "Capacitor_SMD:C_0603_1608Metric"
 			(at 222.25 88.9 0)
 			(effects
@@
 			)
 		)
-		(property "Footprint" ""
+		(property "Footprint" "Resistor_SMD:R_0201_0603Metri"
 			(at 109.22 86.36 0)
 			(effects
@@
 			)
 		)
-		(property "Value" "C"
+		(property "Value" "10uF"
 			(at 172.72 80.0099 0)
 			(effects
@@
 			)
 		)
-		(property "Footprint" ""
+		(property "Footprint" "Capacitor_SMD:C_0603_1608Metric"
 			(at 169.8752 82.55 0)
 			(effects
@@
 	)
 	(symbol
-		(lib_id "Device:D")
-		(at 163.83 71.12 180)
-		(unit 1)
-		(exclude_from_sim no)
-		(in_bom yes)
-		(on_board yes)
-		(dnp no)
-		(fields_autoplaced yes)
-		(property "Reference" "D3"
-			(at 163.83 64.77 0)
-			(effects
-				(font
-					(size 1.27 1.27)
-				)
-			)
-		)
-		(property "Value" "D"
-			(at 163.83 67.31 0)
-			(effects
-				(font
-					(size 1.27 1.27)
-				)
-			)
-		)
-		(property "Footprint" ""
-			(at 163.83 71.12 0)
-			(effects
-				(font
-					(size 1.27 1.27)
-				)
-				(hide yes)
-			)
-		)
-		(property "Datasheet" "~"
-			(at 163.83 71.12 0)
-			(effects
-				(font
-					(size 1.27 1.27)
-				)
-				(hide yes)
-			)
-		)
-		(property "Description" "Diode"
-			(at 163.83 71.12 0)
-			(effects
-				(font
-					(size 1.27 1.27)
-				)
-				(hide yes)
-			)
-		)
-		(property "Sim.Device" "D"
-			(at 163.83 71.12 0)
-			(effects
-				(font
-					(size 1.27 1.27)
-				)
-				(hide yes)
-			)
-		)
-		(property "Sim.Pins" "1=K 2=A"
-			(at 163.83 71.12 0)
-			(effects
-				(font
-					(size 1.27 1.27)
-				)
-				(hide yes)
-			)
-		)
-		(pin "1"
-		)
-		(pin "2"
-		)
-		(instances
-			(project ""
-				(path "/7d0ecb76-dd3a-488e-b45e-ae217463e751/d88ecda6-398d-4f12-9194-bca3a51054e2"
-					(reference "D3")
-					(unit 1)
-				)
-			)
-		)
-	)
-	(symbol
-		(lib_id "Device:D_Zener")
-		(at 270.51 78.74 270)
-		(unit 1)
-		(exclude_from_sim no)
-		(in_bom yes)
-		(on_board yes)
-		(dnp no)
-		(fields_autoplaced yes)
-		(property "Reference" "D5"
-			(at 273.05 77.4699 90)
-			(effects
-				(font
-					(size 1.27 1.27)
-				)
-				(justify left)
-			)
-		)
-		(property "Value" "5V"
-			(at 273.05 80.0099 90)
-			(effects
-				(font
-					(size 1.27 1.27)
-				)
-				(justify left)
-			)
-		)
-		(property "Footprint" ""
-			(at 270.51 78.74 0)
-			(effects
-				(font
-					(size 1.27 1.27)
-				)
-				(hide yes)
-			)
-		)
-		(property "Datasheet" "~"
-			(at 270.51 78.74 0)
-			(effects
-				(font
-					(size 1.27 1.27)
-				)
-				(hide yes)
-			)
-		)
-		(property "Description" "Zener diode"
-			(at 270.51 78.74 0)
-			(effects
-				(font
-					(size 1.27 1.27)
-				)
-				(hide yes)
-			)
-		)
-		(pin "1"
-		)
-		(pin "2"
-		)
-		(instances
-			(project ""
-				(path "/7d0ecb76-dd3a-488e-b45e-ae217463e751/d88ecda6-398d-4f12-9194-bca3a51054e2"
-					(reference "D5")
-					(unit 1)
-				)
-			)
-		)
-	)
-	(symbol
 		(lib_id "power:GND")
 		(at 177.8 86.36 0)
@@
 			)
 		)
-		(property "Footprint" ""
+		(property "Footprint" "Resistor_SMD:R_0201_0603Metri"
 			(at 222.25 82.55 0)
 			(effects
@@
 			)
 		)
-		(property "Value" "470uF"
+		(property "Value" "47uF"
 			(at 262.128 83.058 0)
 			(effects
@@
 			)
 		)
-		(property "Footprint" ""
+		(property "Footprint" "Capacitor_SMD:C_0603_1608Metric"
 			(at 261.3152 82.55 0)
 			(effects
@@
 			)
 		)
-		(property "Footprint" ""
+		(property "Footprint" "Resistor_SMD:R_0201_0603Metri"
 			(at 156.21 74.93 0)
 			(effects
@@
 			)
 		)
-		(property "Footprint" ""
+		(property "Footprint" "Resistor_SMD:R_0201_0603Metri"
 			(at 177.8 74.93 0)
 			(effects
@@
 	)
 	(symbol
+		(lib_id "Diode:BZX84Cxx")
+		(at 270.51 78.74 270)
+		(unit 1)
+		(exclude_from_sim no)
+		(in_bom yes)
+		(on_board yes)
+		(dnp no)
+		(fields_autoplaced yes)
+		(property "Reference" "D3"
+			(at 273.05 77.4699 90)
+			(effects
+				(font
+					(size 1.27 1.27)
+				)
+				(justify left)
+			)
+		)
+		(property "Value" "BZX84W"
+			(at 273.05 80.0099 90)
+			(effects
+				(font
+					(size 1.27 1.27)
+				)
+				(justify left)
+			)
+		)
+		(property "Footprint" "Package_TO_SOT_SMD:SOT-23"
+			(at 270.51 78.74 0)
+			(effects
+				(font
+					(size 1.27 1.27)
+				)
+				(hide yes)
+			)
+		)
+		(property "Datasheet" "https://diotec.com/tl_files/diotec/files/pdf/datasheets/bzx84c2v4.pdf"
+			(at 270.51 78.74 0)
+			(effects
+				(font
+					(size 1.27 1.27)
+				)
+				(hide yes)
+			)
+		)
+		(property "Description" "300mW Zener Diode, SOT-23"
+			(at 270.51 78.74 0)
+			(effects
+				(font
+					(size 1.27 1.27)
+				)
+				(hide yes)
+			)
+		)
+		(pin "3"
+		)
+		(pin "1"
+		)
+		(pin "2"
+		)
+		(instances
+			(project ""
+				(path "/7d0ecb76-dd3a-488e-b45e-ae217463e751/d88ecda6-398d-4f12-9194-bca3a51054e2"
+					(reference "D3")
+					(unit 1)
+				)
+			)
+		)
+	)
+	(symbol
 		(lib_id "Device:R_Small")
 		(at 240.03 82.55 0)
@@
 			)
 		)
-		(property "Footprint" ""
+		(property "Footprint" "Resistor_SMD:R_0201_0603Metri"
 			(at 240.03 82.55 0)
 			(effects
@@
 			)
 		)
-		(property "Footprint" ""
+		(property "Footprint" "Capacitor_SMD:C_0603_1608Metric"
 			(at 81.28 85.09 0)
 			(effects
@@
 			)
 		)
-		(property "Footprint" ""
+		(property "Footprint" "Inductor_SMD:L_12x12mm_H8mm"
 			(at 200.66 60.96 0)
 			(effects
@@
 			)
 		)
-		(property "Footprint" ""
+		(property "Footprint" "Resistor_SMD:R_0201_0603Metri"
 			(at 177.8 82.55 0)
 			(effects
@@
 			)
 		)
-		(property "Footprint" ""
+		(property "Footprint" "Resistor_SMD:R_0201_0603Metri"
 			(at 144.78 74.93 0)
 			(effects
@@
 			)
 		)
-		(property "Footprint" ""
+		(property "Footprint" "Capacitor_SMD:C_0603_1608Metric"
 			(at 250.19 74.93 0)
 			(effects
@@
 			)
 		)
-		(property "Footprint" ""
+		(property "Footprint" "Capacitor_SMD:C_0603_1608Metric"
 			(at 69.85 87.63 0)
 			(effects
@@
 			)
 		)
-		(property "Footprint" ""
+		(property "Footprint" "Resistor_SMD:R_0201_0603Metri"
 			(at 240.03 74.93 0)
 			(effects

Commit message: SCHEMATIC  FINISHED
Parts:
- removed C1: 2.2uF, Capacitor_SMD:C_0603_1608Metric, symbol Device:C_Small
- removed C2: 470pF, Capacitor_SMD:C_0603_1608Metric, symbol Device:C_Small
- removed C8: 47uF, Capacitor_SMD:C_0603_1608Metric, symbol Device:C
- removed U1: MIC5219-3.3YM5, Package_TO_SOT_SMD:SOT-23-5, symbol Regulator_Linear:MIC5219-3.3YM5
- added C1: 470u, symbol Device:C_Polarized
- added C17, C18: 470nF, Capacitor_SMD:C_0603_1608Metric, symbol Device:C_Small
- added J5: Conn_01x02_Socket, symbol Connector:Conn_01x02_Socket
- added U5: BU33SD5WG, Package_TO_SOT_SMD:SOT-23-5, symbol Regulator_Linear:MCP1802x-xx02xOT
- D2: footprint (none) -> LED_SMD:LED_0603_1608Metric
- IC1: MPN (none) -> MIC3172YM; Manufacturer_Part_Number MIC3172YM -> (none)
- L2: value 120uH -> 100uH
- R10, R11, R15, R16, R9: footprint Resistor_SMD:R_0201_0603Metri -> Resistor_SMD:R_0603_1608Metric
- R12: footprint Resistor_SMD:R_0201_0603Metri -> Resistor_SMD:R_0603_1608Metric; MPN (none) -> CRCW06033K74DHEAP
- R13: footprint Resistor_SMD:R_0201_0603Metri -> Resistor_SMD:R_0603_1608Metric; MPN (none) -> CRCW06031K24FKEAHP
- R14: value RISET -> 250R; footprint Resistor_SMD:R_0201_0603Metri -> Resistor_SMD:R_0603_1608Metric
- U4: MPN (none) -> BQ21040DBVR
Connections:
- net -BATT is gone; now on net GND: J4.2 (Pin_2), R9.2, U4.1 (TS)
- net +3.3V: now also C18.1, U5.5 (VOUT)
- net +5V: now also C1.1, C17.1, U5.1 (VIN), U5.3 (~{SHDN})
- net +BATT: now also J5.1 (Pin_1)
- net GND: now also C1.2, C17.2, C18.2, J5.2 (Pin_2), U5.2 (GND)
Other:
- note added: "5V To 3V3 500mA"
- moved on the sheet: U4

Commit message: PCB early
Parts:
- C1: footprint (none) -> Capacitor_SMD:CP_Elec_8x10
- D4: value 1N5822 -> STPS0520Z; footprint Diode_THT:D_DO-201AD_P15.24mm_Horizontal -> Diode_SMD:D_SOD-123
- J4, J5: footprint (none) -> Battery:BatteryHolder_MPD_BH-18650-PC2
Changed lines of the file:
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@@
 			)
 		)
-		(property "Footprint" ""
+		(property "Footprint" "Battery:BatteryHolder_MPD_BH-18650-PC2"
 			(at 212.09 129.54 0)
 			(effects
@@
 			)
 		)
-		(property "Footprint" ""
+		(property "Footprint" "Capacitor_SMD:CP_Elec_8x10"
 			(at 261.3152 82.55 0)
 			(effects
@@
 			)
 		)
-		(property "Footprint" ""
+		(property "Footprint" "Battery:BatteryHolder_MPD_BH-18650-PC2"
 			(at 238.76 129.54 0)
 			(effects
@@
 			)
 		)
-		(property "Value" "1N5822"
+		(property "Value" "STPS0520Z"
 			(at 232.7275 67.31 0)
 			(effects
@@
 			)
 		)
-		(property "Footprint" "Diode_THT:D_DO-201AD_P15.24mm_Horizontal"
+		(property "Footprint" "Diode_SMD:D_SOD-123"
 			(at 232.41 66.675 0)
 			(effects

Commit message: update Alim
Parts:
- IC1: footprint SOIC127P599X173-8N -> MIC3172:SOIC127P599X173-8N
Changed lines of the file:
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@@
 			)
 		)
-		(property "Footprint" "SOIC127P599X173-8N"
+		(property "Footprint" "MIC3172:SOIC127P599X173-8N"
 			(at 215.9 166.04 0)
 			(effects

Commit message: Routing alim
Parts:
- removed C9: 15pf, Capacitor_SMD:C_0603_1608Metric, symbol Device:C_Small
Connections:
- net vsw: now reaches D4.2 (A), IC1.7 (VSW), L2.2
Changed lines of the file:
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@@
 	)
 	(junction
-		(at 240.03 71.12)
-		(diameter 0)
-		(color 0 0 0 0)
-	)
-	(junction
 		(at 34.29 36.83)
 		(diameter 0)
@@
 	)
 	(junction
-		(at 260.35 71.12)
+		(at 270.51 71.12)
 		(diameter 0)
 		(color 0 0 0 0)
 	)
 	(junction
-		(at 270.51 71.12)
+		(at 260.35 71.12)
 		(diameter 0)
 		(color 0 0 0 0)
@@
 	)
 	(junction
-		(at 250.19 71.12)
+		(at 240.03 71.12)
 		(diameter 0)
 		(color 0 0 0 0)
@@
 	(wire
 		(pts
-			(xy 250.19 78.74) (xy 250.19 77.47)
-		)
-		(stroke
-			(width 0)
-			(type default)
-		)
-	)
-	(wire
-		(pts
 			(xy 156.21 86.36) (xy 156.21 90.17)
 		)
@@
 	(wire
 		(pts
-			(xy 250.19 71.12) (xy 260.35 71.12)
+			(xy 240.03 71.12) (xy 260.35 71.12)
 		)
 		(stroke
@@
 	(wire
 		(pts
-			(xy 250.19 71.12) (xy 250.19 72.39)
-		)
-		(stroke
-			(width 0)
-			(type default)
-		)
-	)
-	(wire
-		(pts
 			(xy 177.8 71.12) (xy 177.8 72.39)
 		)
@@
 	(wire
 		(pts
-			(xy 240.03 71.12) (xy 250.19 71.12)
-		)
-		(stroke
-			(width 0)
-			(type default)
-		)
-	)
-	(wire
-		(pts
 			(xy 226.06 74.93) (xy 226.06 78.74)
 		)
@@
 	(wire
 		(pts
-			(xy 240.03 78.74) (xy 250.19 78.74)
+			(xy 144.78 77.47) (xy 144.78 81.28)
 		)
 		(stroke
@@
 		)
 	)
-	(wire
-		(pts
-			(xy 144.78 77.47) (xy 144.78 81.28)
-		)
-		(stroke
-			(width 0)
-			(type default)
+	(label "vsw"
+		(at 220.98 71.12 0)
+		(effects
+			(font
+				(size 1.27 1.27)
+			)
+			(justify left bottom)
 		)
 	)
@@
 					(unit 1)
 				)
-			)
-		)
-	)
-	(symbol
-		(lib_id "Device:C_Small")
-		(at 250.19 74.93 0)
-		(unit 1)
-		(exclude_from_sim no)
-		(in_bom yes)
-		(on_board yes)
-		(dnp no)
-		(property "Reference" "C9"
-			(at 251.714 73.152 0)
-			(effects
-				(font
-					(size 1.27 1.27)
-				)
-				(justify left)
-			)
-		)
-		(property "Value" "15pf"
-			(at 250.19 76.962 0)
-			(effects
-				(font
-					(size 1.27 1.27)
-				)
-				(justify left)
-			)
-		)
-		(property "Footprint" "Capacitor_SMD:C_0603_1608Metric"
-			(at 250.19 74.93 0)
-			(effects
-				(font
-					(size 1.27 1.27)
-				)
-				(hide yes)
-			)
-		)
-		(property "Datasheet" "~"
-			(at 250.19 74.93 0)
-			(effects
-				(font
-					(size 1.27 1.27)
-				)
-				(hide yes)
-			)
-		)
-		(property "Description" "Unpolarized capacitor, small symbol"
-			(at 250.19 74.93 0)
-			(effects
-				(font
-					(size 1.27 1.27)
-				)
-				(hide yes)
-			)
-		)
-		(property "Manufacturer_Part_Number" ""
-			(at 250.19 74.93 0)
-			(effects
-				(font
-					(size 1.27 1.27)
-				)
-			)
-		)
-		(pin "2"
-		)
-		(pin "1"
-		)
-		(instances
-			(project ""
-				(path "/7d0ecb76-dd3a-488e-b45e-ae217463e751/d88ecda6-398d-4f12-9194-bca3a51054e2"
-					(reference "C9")
-					(unit 1)
-				)
