File: Kartrack_Main_Board/CONN.kicad_sch (KiCad schematic)
At the start: 17 parts, among them J1 USB_C_Receptacle_USB2.0_14P, SW1 SW_Push, SW2 SW_Push, SW3 SW_Push

Commit message: PCB early
Parts:
- J1: footprint (none) -> Connector_USB:USB_C_Receptacle_GCT_USB4125-xx-x-0190_6P_TopMnt_Horizontal
Connections:
- net PF8_LORA_RST: now reaches A2.12 (A3)
- no-connect marks 11 -> 10
Changed lines of the file:
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@@
-	)
-	(no_connect
-		(at 201.93 99.06)
 	)
 	(no_connect
@@
 		)
 	)
+	(hierarchical_label "PF8_LORA_RST"
+		(shape input)
+		(at 201.93 99.06 0)
+		(effects
+			(font
+				(size 1.27 1.27)
+			)
+			(justify left)
+		)
+	)
 	(hierarchical_label "PA8"
 		(shape input)
@@
 			)
 		)
-		(property "Footprint" ""
+		(property "Footprint" "Connector_USB:USB_C_Receptacle_GCT_USB4125-xx-x-0190_6P_TopMnt_Horizontal"
 			(at 59.69 90.17 0)
 			(effects
