File: Kartrack_Main_Board/GYRO.kicad_sch (KiCad schematic)
At the start: 3 parts

Commit message: added connectors for pulldown pushbuttons
Parts:
- MT1: footprint ICM-42605:XDCR_ICM-42605 -> ICM-45605:IC_ICM-45605
Changed lines of the file:
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@@
 			)
 		)
-		(property "Footprint" "ICM-42605:XDCR_ICM-42605"
+		(property "Footprint" "ICM-45605:IC_ICM-45605"
 			(at 139.7 95.25 0)
 			(effects

Commit message: update
Parts:
- C14, C15: value 0.1u -> 100nF
Changed lines of the file:
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@@
 			)
 		)
-		(property "Value" "0.1u"
+		(property "Value" "100nF"
 			(at 181.61 81.28 90)
 			(effects
@@
 			)
 		)
-		(property "Value" "0.1u"
+		(property "Value" "100nF"
 			(at 181.61 71.12 90)
 			(effects

Commit message: PCB early
Parts:
- MT1: value ICM-42605 -> ICM-45605
Changed lines of the file:
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@@
 			)
 		)
-		(property "Value" "ICM-42605"
+		(property "Value" "ICM-45605"
 			(at 139.7 80.01 0)
 			(effects
