File: Kartrack_Main_Board/Kartrack_Main_Board.kicad_sch (KiCad schematic)
At the start: 1 part

Commit message: connector
Parts:
- added P1: USB_C_Plug_USB2.0, symbol Connector:USB_C_Plug_USB2.0
Connections:
- new net: P1.A1 (GND), P1.A12 (GND), P1.B1 (GND), P1.B12 (GND)
- new net: P1.A4 (VBUS), P1.A9 (VBUS), P1.B4 (VBUS), P1.B9 (VBUS)
Other:
- added sheet ALIM (ALIM .kicad_sch)
- added sheet CONN (CONN.kicad_sch)
- moved on the sheet: A1
Changed lines of the file:
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@@
 	(paper "A4")
 	(symbol
+		(lib_id "Connector:USB_C_Plug_USB2.0")
+		(at 41.91 111.76 0)
+		(unit 1)
+		(exclude_from_sim no)
+		(in_bom yes)
+		(on_board yes)
+		(dnp no)
+		(fields_autoplaced yes)
+		(property "Reference" "P1"
+			(at 41.91 88.9 0)
+			(effects
+				(font
+					(size 1.27 1.27)
+				)
+			)
+		)
+		(property "Value" "USB_C_Plug_USB2.0"
+			(at 41.91 91.44 0)
+			(effects
+				(font
+					(size 1.27 1.27)
+				)
+			)
+		)
+		(property "Footprint" ""
+			(at 45.72 111.76 0)
+			(effects
+				(font
+					(size 1.27 1.27)
+				)
+				(hide yes)
+			)
+		)
+		(property "Datasheet" "https://www.usb.org/sites/default/files/documents/usb_type-c.zip"
+			(at 45.72 111.76 0)
+			(effects
+				(font
+					(size 1.27 1.27)
+				)
+				(hide yes)
+			)
+		)
+		(property "Description" "USB 2.0-only Type-C Plug connector"
+			(at 41.91 111.76 0)
+			(effects
+				(font
+					(size 1.27 1.27)
+				)
+				(hide yes)
+			)
+		)
+		(pin "A1"
+		)
+		(pin "B4"
+		)
+		(pin "A6"
+		)
+		(pin "B12"
+		)
+		(pin "S1"
+		)
+		(pin "A4"
+		)
+		(pin "B1"
+		)
+		(pin "A9"
+		)
+		(pin "A5"
+		)
+		(pin "A12"
+		)
+		(pin "B5"
+		)
+		(pin "B9"
+		)
+		(pin "A7"
+		)
+		(instances
+			(project ""
+				(path "/7d0ecb76-dd3a-488e-b45e-ae217463e751"
+					(reference "P1")
+					(unit 1)
+				)
+			)
+		)
+	)
+	(symbol
 		(lib_id "MCU_Module:Arduino_UNO_R3")
-		(at 133.35 86.36 0)
+		(at 54.61 45.72 0)
 		(unit 1)
 		(exclude_from_sim no)
@@
 		(fields_autoplaced yes)
 		(property "Reference" "A1"
-			(at 140.5733 58.42 0)
+			(at 61.8333 17.78 0)
 			(effects
 				(font
@@
 		)
 		(property "Value" "Arduino_UNO_R3"
-			(at 140.5733 60.96 0)
+			(at 61.8333 20.32 0)
 			(effects
 				(font
@@
 		)
 		(property "Footprint" "Module:Arduino_UNO_R3"
-			(at 133.35 86.36 0)
+			(at 54.61 45.72 0)
 			(effects
 				(font
@@
 		)
 		(property "Datasheet" "https://www.arduino.cc/en/Main/arduinoBoardUno"
-			(at 133.35 86.36 0)
+			(at 54.61 45.72 0)
 			(effects
 				(font
@@
 		)
 		(property "Description" "Arduino UNO Microcontroller Module, release 3"
-			(at 133.35 86.36 0)
+			(at 54.61 45.72 0)
 			(effects
 				(font
@@
 				)
 			)
+		)
+	)
+	(sheet
+		(at 212.09 64.77)
+		(size 27.94 34.29)
+		(exclude_from_sim no)
+		(in_bom yes)
+		(on_board yes)
+		(dnp no)
+		(fields_autoplaced yes)
+		(stroke
+			(width 0.1524)
+			(type solid)
+		)
+		(fill
+			(color 0 0 0 0.0000)
+		)
+		(property "Sheetname" "CONN"
+			(at 212.09 64.0584 0)
+			(effects
+				(font
+					(size 1.27 1.27)
+				)
+				(justify left bottom)
+			)
+		)
+		(property "Sheetfile" "CONN.kicad_sch"
+			(at 212.09 99.6446 0)
+			(effects
+				(font
+					(size 1.27 1.27)
+				)
+				(justify left top)
+			)
+		)
+		(instances
+			(project "Kartrack_Main_Board"
+				(path "/7d0ecb76-dd3a-488e-b45e-ae217463e751"
+					(page "3")
+				)
+			)
+		)
+	)
+	(sheet
+		(at 148.59 63.5)
+		(size 38.1 46.99)
+		(exclude_from_sim no)
+		(in_bom yes)
+		(on_board yes)
+		(dnp no)
+		(fields_autoplaced yes)
+		(stroke
+			(width 0.1524)
+			(type solid)
+		)
+		(fill
+			(color 0 0 0 0.0000)
+		)
+		(property "Sheetname" "ALIM"
+			(at 148.59 62.7884 0)
+			(effects
+				(font
+					(size 1.27 1.27)
+				)
+				(justify left bottom)
+			)
+		)
+		(property "Sheetfile" "ALIM .kicad_sch"
+			(at 148.59 111.0746 0)
+			(effects
+				(font
+					(size 1.27 1.27)
+				)
+				(justify left top)
+			)
+		)
+		(instances
+			(project "Kartrack_Main_Board"
+				(path "/7d0ecb76-dd3a-488e-b45e-ae217463e751"
+					(page "2")
+				)
+			)

Commit message: schematic GPS
Parts:
- removed A1: Arduino_UNO_R3, Module:Arduino_UNO_R3, symbol MCU_Module:Arduino_UNO_R3
- removed P1: USB_C_Plug_USB2.0, symbol Connector:USB_C_Plug_USB2.0
Other:
- added sheet GPS (GPS.kicad_sch)
Changed lines of the file:
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@@
 	(generator_version "9.0")
 	(paper "A4")
-	(symbol
-		(lib_id "Connector:USB_C_Plug_USB2.0")
-		(at 41.91 111.76 0)
-		(unit 1)
-		(exclude_from_sim no)
-		(in_bom yes)
-		(on_board yes)
-		(dnp no)
-		(fields_autoplaced yes)
-		(property "Reference" "P1"
-			(at 41.91 88.9 0)
-			(effects
-				(font
-					(size 1.27 1.27)
-				)
-			)
-		)
-		(property "Value" "USB_C_Plug_USB2.0"
-			(at 41.91 91.44 0)
-			(effects
-				(font
-					(size 1.27 1.27)
-				)
-			)
-		)
-		(property "Footprint" ""
-			(at 45.72 111.76 0)
-			(effects
-				(font
-					(size 1.27 1.27)
-				)
-				(hide yes)
-			)
-		)
-		(property "Datasheet" "https://www.usb.org/sites/default/files/documents/usb_type-c.zip"
-			(at 45.72 111.76 0)
-			(effects
-				(font
-					(size 1.27 1.27)
-				)
-				(hide yes)
-			)
-		)
-		(property "Description" "USB 2.0-only Type-C Plug connector"
-			(at 41.91 111.76 0)
-			(effects
-				(font
-					(size 1.27 1.27)
-				)
-				(hide yes)
-			)
-		)
-		(pin "A1"
-		)
-		(pin "B4"
-		)
-		(pin "A6"
-		)
-		(pin "B12"
-		)
-		(pin "S1"
-		)
-		(pin "A4"
-		)
-		(pin "B1"
-		)
-		(pin "A9"
-		)
-		(pin "A5"
-		)
-		(pin "A12"
-		)
-		(pin "B5"
-		)
-		(pin "B9"
-		)
-		(pin "A7"
-		)
-		(instances
-			(project ""
-				(path "/7d0ecb76-dd3a-488e-b45e-ae217463e751"
-					(reference "P1")
-					(unit 1)
-				)
-			)
-		)
-	)
-	(symbol
-		(lib_id "MCU_Module:Arduino_UNO_R3")
-		(at 54.61 45.72 0)
-		(unit 1)
-		(exclude_from_sim no)
-		(in_bom yes)
-		(on_board yes)
-		(dnp no)
-		(fields_autoplaced yes)
-		(property "Reference" "A1"
-			(at 61.8333 17.78 0)
-			(effects
-				(font
-					(size 1.27 1.27)
-				)
-				(justify left)
-			)
-		)
-		(property "Value" "Arduino_UNO_R3"
-			(at 61.8333 20.32 0)
-			(effects
-				(font
-					(size 1.27 1.27)
-				)
-				(justify left)
-			)
-		)
-		(property "Footprint" "Module:Arduino_UNO_R3"
-			(at 54.61 45.72 0)
-			(effects
-				(font
-					(size 1.27 1.27)
-					(italic yes)
-				)
-				(hide yes)
-			)
-		)
-		(property "Datasheet" "https://www.arduino.cc/en/Main/arduinoBoardUno"
-			(at 54.61 45.72 0)
-			(effects
-				(font
-					(size 1.27 1.27)
-				)
-				(hide yes)
-			)
-		)
-		(property "Description" "Arduino UNO Microcontroller Module, release 3"
-			(at 54.61 45.72 0)
-			(effects
-				(font
-					(size 1.27 1.27)
-				)
-				(hide yes)
-			)
-		)
-		(pin "10"
-		)
-		(pin "25"
-		)
-		(pin "26"
-		)
-		(pin "17"
-		)
-		(pin "28"
-		)
-		(pin "18"
-		)
-		(pin "32"
-		)
-		(pin "27"
-		)
-		(pin "23"
-		)
-		(pin "22"
-		)
-		(pin "20"
-		)
-		(pin "21"
-		)
-		(pin "16"
-		)
-		(pin "15"
-		)
-		(pin "6"
-		)
-		(pin "4"
-		)
-		(pin "24"
-		)
-		(pin "5"
-		)
-		(pin "9"
-		)
-		(pin "3"
-		)
-		(pin "2"
-		)
-		(pin "19"
-		)
-		(pin "13"
-		)
-		(pin "12"
-		)
-		(pin "31"
-		)
-		(pin "1"
-		)
-		(pin "14"
-		)
-		(pin "29"
-		)
-		(pin "11"
-		)
-		(pin "8"
-		)
-		(pin "30"
-		)
-		(pin "7"
-		)
-		(instances
-			(project ""
-				(path "/7d0ecb76-dd3a-488e-b45e-ae217463e751"
-					(reference "A1")
-					(unit 1)
-				)
-			)
-		)
-	)
 	(sheet
 		(at 212.09 64.77)
@@
 				)
 			)
+		)
+	)
+	(sheet
+		(at 49.53 58.42)
+		(size 24.13 24.13)
+		(exclude_from_sim no)
+		(in_bom yes)
+		(on_board yes)
+		(dnp no)
+		(fields_autoplaced yes)
+		(stroke
+			(width 0.1524)
+			(type solid)
+		)
+		(fill
+			(color 0 0 0 0.0000)
+		)
+		(property "Sheetname" "GPS"
+			(at 49.53 57.7084 0)
+			(effects
+				(font
+					(size 1.27 1.27)
+				)
+				(justify left bottom)
+			)
+		)
+		(property "Sheetfile" "GPS.kicad_sch"
+			(at 49.53 83.1346 0)
+			(effects
+				(font
+					(size 1.27 1.27)
+				)
+				(justify left top)
+			)
+		)
+		(instances
+			(project "Kartrack_Main_Board"
+				(path "/7d0ecb76-dd3a-488e-b45e-ae217463e751"
+					(page "4")
+				)
+			)

Commit message: Schematic
Other:
- added sheet GYRO (GYRO.kicad_sch)
- added sheet LORA (LORA.kicad_sch)
- sheet GPS ports: added RX_GPS, TX_GSP; removed none
Changed lines of the file:
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@@
 	(paper "A4")
+	(sheet
+		(at 29.21 27.94)
+		(size 19.05 20.32)
+		(exclude_from_sim no)
+		(in_bom yes)
+		(on_board yes)
+		(dnp no)
+		(fields_autoplaced yes)
+		(stroke
+			(width 0.1524)
+			(type solid)
+		)
+		(fill
+			(color 0 0 0 0.0000)
+		)
+		(property "Sheetname" "LORA"
+			(at 29.21 27.2284 0)
+			(effects
+				(font
+					(size 1.27 1.27)
+				)
+				(justify left bottom)
+			)
+		)
+		(property "Sheetfile" "LORA.kicad_sch"
+			(at 29.21 48.8446 0)
+			(effects
+				(font
+					(size 1.27 1.27)
+				)
+				(justify left top)
+			)
+		)
+		(pin "SCK" input
+			(at 48.26 31.75 0)
+			(effects
+				(font
+					(size 1.27 1.27)
+				)
+				(justify right)
+			)
+		)
+		(pin "{slash}NSS" input
+			(at 48.26 35.56 0)
+			(effects
+				(font
+					(size 1.27 1.27)
+				)
+				(justify right)
+			)
+		)
+		(pin "MOSI" input
+			(at 48.26 39.37 0)
+			(effects
+				(font
+					(size 1.27 1.27)
+				)
+				(justify right)
+			)
+		)
+		(pin "MISO" input
+			(at 48.26 43.18 0)
+			(effects
+				(font
+					(size 1.27 1.27)
+				)
+				(justify right)
+			)
+		)
+		(instances
+			(project "Kartrack_Main_Board"
+				(path "/7d0ecb76-dd3a-488e-b45e-ae217463e751"
+					(page "6")
+				)
+			)
+		)
+	)
+	(sheet
+		(at 26.67 102.87)
+		(size 33.02 30.48)
+		(exclude_from_sim no)
+		(in_bom yes)
+		(on_board yes)
+		(dnp no)
+		(fields_autoplaced yes)
+		(stroke
+			(width 0.1524)
+			(type solid)
+		)
+		(fill
+			(color 0 0 0 0.0000)
+		)
+		(property "Sheetname" "GYRO"
+			(at 26.67 102.1584 0)
+			(effects
+				(font
+					(size 1.27 1.27)
+				)
+				(justify left bottom)
+			)
+		)
+		(property "Sheetfile" "GYRO.kicad_sch"
+			(at 26.67 133.9346 0)
+			(effects
+				(font
+					(size 1.27 1.27)
+				)
+				(justify left top)
+			)
+		)
+		(pin "i2c1_SCL" input
+			(at 59.69 110.49 0)
+			(effects
+				(font
+					(size 1.27 1.27)
+				)
+				(justify right)
+			)
+		)
+		(pin "Gyro_IT1" input
+			(at 59.69 124.46 0)
+			(effects
+				(font
+					(size 1.27 1.27)
+				)
+				(justify right)
+			)
+		)
+		(pin "Gyro_IT2" input
+			(at 59.69 128.27 0)
+			(effects
+				(font
+					(size 1.27 1.27)
+				)
+				(justify right)
+			)
+		)
+		(pin "i2c1_SDA" input
+			(at 59.69 113.03 0)
+			(effects
+				(font
+					(size 1.27 1.27)
+				)
+				(justify right)
+			)
+		)
+		(instances
+			(project "Kartrack_Main_Board"
+				(path "/7d0ecb76-dd3a-488e-b45e-ae217463e751"
+					(page "5")
+				)
+			)
+		)
+	)
 	(sheet
 		(at 212.09 64.77)
@@
 	)
 	(sheet
-		(at 148.59 63.5)
-		(size 38.1 46.99)
+		(at 242.57 30.48)
+		(size 25.4 22.86)
 		(exclude_from_sim no)
 		(in_bom yes)
@@
 		)
 		(property "Sheetname" "ALIM"
-			(at 148.59 62.7884 0)
+			(at 242.57 29.7684 0)
 			(effects
 				(font
@@
 		)
 		(property "Sheetfile" "ALIM .kicad_sch"
-			(at 148.59 111.0746 0)
+			(at 242.57 53.9246 0)
 			(effects
 				(font
@@
 	)
 	(sheet
-		(at 49.53 58.42)
+		(at 26.67 55.88)
 		(size 24.13 24.13)
 		(exclude_from_sim no)
@@
 		)
 		(property "Sheetname" "GPS"
-			(at 49.53 57.7084 0)
+			(at 26.67 55.1684 0)
 			(effects
 				(font
@@
 		)
 		(property "Sheetfile" "GPS.kicad_sch"
-			(at 49.53 83.1346 0)
-			(effects
-				(font
-					(size 1.27 1.27)
-				)
-				(justify left top)
-			)
-		)
+			(at 26.67 80.5946 0)
+			(effects
+				(font
+					(size 1.27 1.27)
+				)
+				(justify left top)
+			)
+		)
+		(pin "RX_GPS" input
+			(at 50.8 62.23 0)
+			(effects
+				(font
+					(size 1.27 1.27)
+				)
+				(justify right)
+			)
+		)
+		(pin "TX_GSP" input
+			(at 50.8 69.85 0)
+			(effects
+				(font
+					(size 1.27 1.27)
+				)
+				(justify right)
+			)
+		)

Commit message: FIn de séance
Changed lines of the file:
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@@
 	(paper "A4")
 	(sheet
-		(at 29.21 27.94)
+		(at 128.27 25.4)
 		(size 19.05 20.32)
 		(exclude_from_sim no)
@@
 		)
 		(property "Sheetname" "LORA"
-			(at 29.21 27.2284 0)
+			(at 128.27 24.6884 0)
 			(effects
 				(font
@@
 		)
 		(property "Sheetfile" "LORA.kicad_sch"
-			(at 29.21 48.8446 0)
+			(at 128.27 46.3046 0)
 			(effects
 				(font
@@
 		)
 		(pin "SCK" input
-			(at 48.26 31.75 0)
+			(at 147.32 29.21 0)
 			(effects
 				(font
@@
 		)
 		(pin "{slash}NSS" input
-			(at 48.26 35.56 0)
+			(at 147.32 33.02 0)
 			(effects
 				(font
@@
 		)
 		(pin "MOSI" input
-			(at 48.26 39.37 0)
+			(at 147.32 36.83 0)
 			(effects
 				(font
@@
 		)
 		(pin "MISO" input
-			(at 48.26 43.18 0)
+			(at 147.32 40.64 0)
 			(effects
 				(font
@@
 	)
 	(sheet
-		(at 26.67 102.87)
+		(at 128.27 90.17)
 		(size 33.02 30.48)
 		(exclude_from_sim no)
@@
 		)
 		(property "Sheetname" "GYRO"
-			(at 26.67 102.1584 0)
+			(at 128.27 89.4584 0)
 			(effects
 				(font
@@
 		)
 		(property "Sheetfile" "GYRO.kicad_sch"
-			(at 26.67 133.9346 0)
+			(at 128.27 121.2346 0)
 			(effects
 				(font
@@
 		)
 		(pin "i2c1_SCL" input
-			(at 59.69 110.49 0)
+			(at 161.29 97.79 0)
 			(effects
 				(font
@@
 		)
 		(pin "Gyro_IT1" input
-			(at 59.69 124.46 0)
+			(at 161.29 111.76 0)
 			(effects
 				(font
@@
 		)
 		(pin "Gyro_IT2" input
-			(at 59.69 128.27 0)
+			(at 161.29 115.57 0)
 			(effects
 				(font
@@
 		)
 		(pin "i2c1_SDA" input
-			(at 59.69 113.03 0)
+			(at 161.29 100.33 0)
 			(effects
 				(font
@@
 	)
 	(sheet
-		(at 212.09 64.77)
+		(at 241.3 80.01)
 		(size 27.94 34.29)
 		(exclude_from_sim no)
@@
 		)
 		(property "Sheetname" "CONN"
-			(at 212.09 64.0584 0)
+			(at 241.3 79.2984 0)
 			(effects
 				(font
@@
 		)
 		(property "Sheetfile" "CONN.kicad_sch"
-			(at 212.09 99.6446 0)
+			(at 241.3 114.8846 0)
 			(effects
 				(font
@@
 	)
 	(sheet
-		(at 242.57 30.48)
+		(at 133.35 129.54)
 		(size 25.4 22.86)
 		(exclude_from_sim no)
@@
 		)
 		(property "Sheetname" "ALIM"
-			(at 242.57 29.7684 0)
+			(at 133.35 128.8284 0)
 			(effects
 				(font
@@
 		)
 		(property "Sheetfile" "ALIM .kicad_sch"
-			(at 242.57 53.9246 0)
+			(at 133.35 152.9846 0)
 			(effects
 				(font
@@
 	)
 	(sheet
-		(at 26.67 55.88)
+		(at 129.54 55.88)
 		(size 24.13 24.13)
 		(exclude_from_sim no)
@@
 		)
 		(property "Sheetname" "GPS"
-			(at 26.67 55.1684 0)
+			(at 129.54 55.1684 0)
 			(effects
 				(font
@@
 		)
 		(property "Sheetfile" "GPS.kicad_sch"
-			(at 26.67 80.5946 0)
+			(at 129.54 80.5946 0)
 			(effects
 				(font
@@
 		)
 		(pin "RX_GPS" input
-			(at 50.8 62.23 0)
+			(at 153.67 62.23 0)
 			(effects
 				(font
@@
 		)
 		(pin "TX_GSP" input
-			(at 50.8 69.85 0)
-			(effects
-				(font
+			(at 153.67 69.85 0)
+			(effects
+				(font

Commit message: BLOC schematic
Other:
- sheet CONN ports: added NRESET, PA15, PA8, PB14_SPI2_MISO, PB15_SPI2_MOSI, PB4, PB8_SCL, PB9_SDA, PC6_TX, PC7_RX, PG6, PG7, PI1_SPI2_SCK, PI2, PI3, PIO_SPI2_NSS; removed none
- sheet LORA ports: added DIO0, DIO1, DIO2, DIO3, DIO4, DIO5; removed none

Commit message: update
Other:
- sheet LORA ports: added none; removed DIO5
Changed lines of the file:
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@@
 	(wire
 		(pts
-			(xy 147.32 45.72) (xy 190.5 45.72)
+			(xy 147.32 45.72) (xy 193.04 45.72)
 		)
 		(stroke
@@
 	(wire
 		(pts
-			(xy 199.39 73.66) (xy 241.3 73.66)
-		)
-		(stroke
-			(width 0)
-			(type default)
-		)
-	)
-	(wire
-		(pts
-			(xy 157.48 104.14) (xy 241.3 104.14)
+			(xy 200.66 73.66) (xy 241.3 73.66)
+		)
+		(stroke
+			(width 0)
+			(type default)
+		)
+	)
+	(wire
+		(pts
+			(xy 158.75 104.14) (xy 241.3 104.14)
 		)
 		(stroke
@@
 	(wire
 		(pts
-			(xy 157.48 83.82) (xy 157.48 104.14)
-		)
-		(stroke
-			(width 0)
-			(type default)
-		)
-	)
-	(wire
-		(pts
-			(xy 195.58 76.2) (xy 195.58 40.64)
+			(xy 158.75 83.82) (xy 158.75 104.14)
+		)
+		(stroke
+			(width 0)
+			(type default)
+		)
+	)
+	(wire
+		(pts
+			(xy 198.12 76.2) (xy 198.12 40.64)
 		)
 		(stroke
@@
 	(wire
 		(pts
-			(xy 151.13 66.04) (xy 166.37 66.04)
-		)
-		(stroke
-			(width 0)
-			(type default)
-		)
-	)
-	(wire
-		(pts
-			(xy 151.13 83.82) (xy 157.48 83.82)
+			(xy 151.13 66.04) (xy 167.64 66.04)
+		)
+		(stroke
+			(width 0)
+			(type default)
+		)
+	)
+	(wire
+		(pts
+			(xy 151.13 83.82) (xy 158.75 83.82)
 		)
 		(stroke
@@
 	(wire
 		(pts
-			(xy 190.5 45.72) (xy 190.5 81.28)
-		)
-		(stroke
-			(width 0)
-			(type default)
-		)
-	)
-	(wire
-		(pts
-			(xy 187.96 83.82) (xy 241.3 83.82)
+			(xy 193.04 45.72) (xy 193.04 81.28)
+		)
+		(stroke
+			(width 0)
+			(type default)
+		)
+	)
+	(wire
+		(pts
+			(xy 190.5 83.82) (xy 241.3 83.82)
 		)
 		(stroke
@@
 	(wire
 		(pts
-			(xy 147.32 38.1) (xy 199.39 38.1)
-		)
-		(stroke
-			(width 0)
-			(type default)
-		)
-	)
-	(wire
-		(pts
-			(xy 166.37 99.06) (xy 241.3 99.06)
+			(xy 147.32 38.1) (xy 200.66 38.1)
+		)
+		(stroke
+			(width 0)
+			(type default)
+		)
+	)
+	(wire
+		(pts
+			(xy 167.64 99.06) (xy 241.3 99.06)
 		)
 		(stroke
@@
 	(wire
 		(pts
-			(xy 199.39 38.1) (xy 199.39 73.66)
-		)
-		(stroke
-			(width 0)
-			(type default)
-		)
-	)
-	(wire
-		(pts
-			(xy 147.32 48.26) (xy 187.96 48.26)
+			(xy 200.66 38.1) (xy 200.66 73.66)
+		)
+		(stroke
+			(width 0)
+			(type default)
+		)
+	)
+	(wire
+		(pts
+			(xy 147.32 48.26) (xy 190.5 48.26)
 		)
 		(stroke
@@
 	(wire
 		(pts
-			(xy 187.96 48.26) (xy 187.96 83.82)
+			(xy 190.5 48.26) (xy 190.5 83.82)
 		)
 		(stroke
@@
 	(wire
 		(pts
-			(xy 195.58 76.2) (xy 241.3 76.2)
-		)
-		(stroke
-			(width 0)
-			(type default)
-		)
-	)
-	(wire
-		(pts
-			(xy 190.5 81.28) (xy 241.3 81.28)
-		)
-		(stroke
-			(width 0)
-			(type default)
-		)
-	)
-	(wire
-		(pts
-			(xy 193.04 78.74) (xy 241.3 78.74)
-		)
-		(stroke
-			(width 0)
-			(type default)
-		)
-	)
-	(wire
-		(pts
-			(xy 166.37 66.04) (xy 166.37 99.06)
-		)
-		(stroke
-			(width 0)
-			(type default)
-		)
-	)
-	(wire
-		(pts
-			(xy 147.32 43.18) (xy 193.04 43.18)
-		)
-		(stroke
-			(width 0)
-			(type default)
-		)
-	)
-	(wire
-		(pts
-			(xy 147.32 40.64) (xy 195.58 40.64)
+			(xy 198.12 76.2) (xy 241.3 76.2)
+		)
+		(stroke
+			(width 0)
+			(type default)
+		)
+	)
+	(wire
+		(pts
+			(xy 193.04 81.28) (xy 241.3 81.28)
+		)
+		(stroke
+			(width 0)
+			(type default)
+		)
+	)
+	(wire
+		(pts
+			(xy 195.58 78.74) (xy 241.3 78.74)
+		)
+		(stroke
+			(width 0)
+			(type default)
+		)
+	)
+	(wire
+		(pts
+			(xy 167.64 66.04) (xy 167.64 99.06)
+		)
+		(stroke
+			(width 0)
+			(type default)
+		)
+	)
+	(wire
+		(pts
+			(xy 147.32 43.18) (xy 195.58 43.18)
+		)
+		(stroke
+			(width 0)
+			(type default)
+		)
+	)
+	(wire
+		(pts
+			(xy 147.32 40.64) (xy 198.12 40.64)
 		)
 		(stroke
@@
 	(wire
 		(pts
-			(xy 193.04 43.18) (xy 193.04 78.74)
+			(xy 195.58 43.18) (xy 195.58 78.74)
 		)
 		(stroke
@@
 			(effects
 				(font
-					(size 1.27 1.27)
-				)
-				(justify right)
-			)
-		)
-		(pin "DIO5" input
-			(at 147.32 50.8 0)
-			(effects
-				(font

Commit message: SCHEMATIC  FINISHED
Other:
- sheet CONN ports: added PF6_STBY_GPS; removed NRESET
- sheet GPS ports: added STBY_GPS; removed none
Changed lines of the file:
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@@
+	(wire
+		(pts
+			(xy 140.97 106.68) (xy 241.3 106.68)
+		)
+		(stroke
+			(width 0)
+			(type default)
+		)
+	)
 	(wire
 		(pts
@@
 			)
 		)
-		(pin "NRESET" input
-			(at 269.24 83.82 0)
-			(effects
-				(font
-					(size 1.27 1.27)
-				)
-				(justify right)
-			)
-		)
 		(pin "PB9_SDA" input
 			(at 241.3 96.52 180)
@@
 		(pin "PB4" input
 			(at 241.3 83.82 180)
+			(effects
+				(font
+					(size 1.27 1.27)
+				)
+				(justify left)
+			)
+		)
+		(pin "PF6_STBY_GPS" input
+			(at 241.3 106.68 180)
 			(effects
 				(font
@@
 			(effects
 				(font
+					(size 1.27 1.27)
+				)
+				(justify right)
+			)
+		)
+		(pin "STBY_GPS" input
+			(at 140.97 106.68 0)
+			(effects
+				(font

Commit message: PCB early
Other:
- sheet CONN ports: added PF8_LORA_RST; removed none
- sheet LORA ports: added RST; removed none
Changed lines of the file:
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@@
+	(wire
+		(pts
+			(xy 147.32 50.8) (xy 187.96 50.8)
+		)
+		(stroke
+			(width 0)
+			(type default)
+		)
+	)
 	(wire
 		(pts
@@
 	(wire
 		(pts
+			(xy 187.96 50.8) (xy 187.96 86.36)
+		)
+		(stroke
+			(width 0)
+			(type default)
+		)
+	)
+	(wire
+		(pts
 			(xy 210.82 27.94) (xy 210.82 63.5)
 		)
@@
 		(pts
 			(xy 147.32 48.26) (xy 190.5 48.26)
+		)
+		(stroke
+			(width 0)
+			(type default)
+		)
+	)
+	(wire
+		(pts
+			(xy 187.96 86.36) (xy 241.3 86.36)
 		)
 		(stroke
@@
 			)
 		)
+		(pin "RST" input
+			(at 147.32 50.8 0)
+			(effects
+				(font
+					(size 1.27 1.27)
+				)
+				(justify right)
+			)
+		)
 		(instances
 			(project "Kartrack_Main_Board"
@@
 			(effects
 				(font
+					(size 1.27 1.27)
+				)
+				(justify left)
+			)
+		)
+		(pin "PF8_LORA_RST" input
+			(at 241.3 86.36 180)
+			(effects
+				(font
