File: Kartrack_Main_Board/GPS.kicad_sch (KiCad schematic)
At the start: 20 parts, among them J2 Conn_Coaxial, Q1 S8050, U2 L76L-M33

Commit message: Schematic
Other:
- moved on the sheet: JP6, U2

Commit message: BLOC schematic
Parts:
- added R17, R18: 0, symbol Device:R_Small
Connections:
- net RX_GPS: now also R17.2; no longer U2.3 (RXD1)
- net TX_GSP: now also R18.2; no longer U2.2 (TXD1)
- new net: R17.1, U2.3 (RXD1)
- new net: R18.1, U2.2 (TXD1)
Changed lines of the file:
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@@
+	(wire
+		(pts
+			(xy 214.63 101.6) (xy 210.82 101.6)
+		)
+		(stroke
+			(width 0)
+			(type default)
+		)
+	)
 	(wire
 		(pts
@@
 	(wire
 		(pts
+			(xy 205.74 101.6) (xy 203.2 101.6)
+		)
+		(stroke
+			(width 0)
+			(type default)
+		)
+	)
+	(wire
+		(pts
 			(xy 40.64 55.88) (xy 45.72 55.88)
 		)
@@
 	(wire
 		(pts
+			(xy 214.63 99.06) (xy 210.82 99.06)
+		)
+		(stroke
+			(width 0)
+			(type default)
+		)
+	)
+	(wire
+		(pts
 			(xy 110.49 36.83) (xy 115.57 36.83)
 		)
@@
 		(pts
 			(xy 158.75 99.06) (xy 162.56 99.06)
+		)
+		(stroke
+			(width 0)
+			(type default)
+		)
+	)
+	(wire
+		(pts
+			(xy 205.74 99.06) (xy 203.2 99.06)
 		)
 		(stroke
@@
 	(hierarchical_label "TX_GSP"
 		(shape input)
-		(at 203.2 101.6 0)
+		(at 214.63 101.6 0)
 		(effects
 			(font
@@
 	(hierarchical_label "RX_GPS"
 		(shape input)
-		(at 203.2 99.06 0)
+		(at 214.63 99.06 0)
 		(effects
 			(font
@@
 	)
 	(symbol
+		(lib_id "Device:R_Small")
+		(at 208.28 99.06 90)
+		(unit 1)
+		(exclude_from_sim no)
+		(in_bom yes)
+		(on_board yes)
+		(dnp no)
+		(fields_autoplaced yes)
+		(property "Reference" "R17"
+			(at 208.28 93.98 90)
+			(effects
+				(font
+					(size 1.27 1.27)
+				)
+			)
+		)
+		(property "Value" "0"
+			(at 208.28 96.52 90)
+			(effects
+				(font
+					(size 1.27 1.27)
+				)
+			)
+		)
+		(property "Footprint" ""
+			(at 208.28 99.06 0)
+			(effects
+				(font
+					(size 1.27 1.27)
+				)
+				(hide yes)
+			)
+		)
+		(property "Datasheet" "~"
+			(at 208.28 99.06 0)
+			(effects
+				(font
+					(size 1.27 1.27)
+				)
+				(hide yes)
+			)
+		)
+		(property "Description" "Resistor, small symbol"
+			(at 208.28 99.06 0)
+			(effects
+				(font
+					(size 1.27 1.27)
+				)
+				(hide yes)
+			)
+		)
+		(pin "1"
+		)
+		(pin "2"
+		)
+		(instances
+			(project ""
+				(path "/7d0ecb76-dd3a-488e-b45e-ae217463e751/f4057792-7e82-430d-87ae-79f44558fd95"
+					(reference "R17")
+					(unit 1)
+				)
+			)
+		)
+	)
+	(symbol
 		(lib_id "power:GND")
 		(at 40.64 115.57 0)
@@
 					(unit 1)
 				)
+			)
+		)
+	)
+	(symbol
+		(lib_id "Device:R_Small")
+		(at 208.28 101.6 90)
+		(unit 1)
+		(exclude_from_sim no)
+		(in_bom yes)
+		(on_board yes)
+		(dnp no)
+		(property "Reference" "R18"
+			(at 208.28 105.156 90)
+			(effects
+				(font
+					(size 1.27 1.27)
+				)
+			)
+		)
+		(property "Value" "0"
+			(at 208.28 103.632 90)
+			(effects
+				(font
+					(size 1.27 1.27)
+				)
+			)
+		)
+		(property "Footprint" ""
+			(at 208.28 101.6 0)
+			(effects
+				(font
+					(size 1.27 1.27)
+				)
+				(hide yes)
+			)
+		)
+		(property "Datasheet" "~"
+			(at 208.28 101.6 0)
+			(effects
+				(font
+					(size 1.27 1.27)
+				)
+				(hide yes)
+			)
+		)
+		(property "Description" "Resistor, small symbol"
+			(at 208.28 101.6 0)
+			(effects
+				(font
+					(size 1.27 1.27)
+				)
+				(hide yes)
+			)
+		)
+		(pin "1"
+		)
+		(pin "2"
+		)
+		(instances
+			(project "Kartrack_Main_Board"
+				(path "/7d0ecb76-dd3a-488e-b45e-ae217463e751/f4057792-7e82-430d-87ae-79f44558fd95"
+					(reference "R18")
+					(unit 1)
+				)

Commit message: update
Parts:
- removed D1: D_Zener, symbol Device:D_Zener
- added C11: 100pF, Capacitor_SMD:C_0603_1608Metric, symbol Device:C
- added D1: 1N4148WS, Diode_SMD:D_SOD-323, symbol Diode:1N4148WS
- added R22: 100R, Resistor_SMD:R_0201_0603Metri, symbol Device:R_Small
- C3: value C -> 100nF; footprint (none) -> Capacitor_SMD:C_0603_1608Metric
- C4: value C -> 10uF; footprint (none) -> Capacitor_SMD:C_0603_1608Metric
- C5, C6: footprint (none) -> Capacitor_SMD:C_0603_1608Metric
- L1: footprint (none) -> Inductor_SMD:L_0603_1608Metric
- R17, R18, R3, R4, R5, R6, R7, R8: footprint (none) -> Resistor_SMD:R_0201_0603Metri
Connections:
- net RF_IN: now also C11.2; no longer J2.1 (In), L1.2
- net VCC_RF: now also R22.2; no longer U2.14 (VCC_RF)
- net at JP4.1 (A), JP5.1 (A): now also D1.2 (A)
- net at R6.1: now also D1.1 (K)
- new net: R22.1, U2.14 (VCC_RF)
- new net: C11.1, J2.1 (In), L1.2
Other:
- moved on the sheet: C5, C6

Commit message: SCHEMATIC  FINISHED
Parts:
- removed JP3, JP4, JP5: SolderJumper_2_Open, symbol Jumper:SolderJumper_2_Open
- added R19: 0, Resistor_SMD:R_0603_1608Metric, symbol Device:R_Small
- Q1: footprint Package_TO_SOT_THT:TO-92_Inline -> Resistor_SMD:R_0603_1608Metric
- R17, R18, R22, R3, R4, R5, R6, R7, R8: footprint Resistor_SMD:R_0201_0603Metri -> Resistor_SMD:R_0603_1608Metric
Connections:
- net +3.3V: now also R19.2
- net STBY_GPS: now reaches D1.2 (A)
- net +3.3V_GPS: no longer names the net of C3.1, C4.1
- net +3.3V_GPS: no longer JP2.2 (B), U2.8 (VCC)
- net VCC_RF: no longer names the net of R22.2
- net VCC_RF: no longer L1.1
Other:
- moved on the sheet: JP2, R3, R4, R5

Commit message: PCB early
Parts:
- J2: footprint (none) -> Connector_Coaxial:U.FL_Molex_MCRF_73412-0110_Vertical
- Q1: value S8050 -> RE1C; footprint Resistor_SMD:R_0603_1608Metric -> Package_TO_SOT_SMD:SOT-416; now left out of the parts list
Changed lines of the file:
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@@
 			)
 		)
-		(property "Footprint" ""
+		(property "Footprint" "Connector_Coaxial:U.FL_Molex_MCRF_73412-0110_Vertical"
 			(at 40.64 102.87 0)
 			(effects
@@
 		(unit 1)
 		(exclude_from_sim no)
-		(in_bom yes)
+		(in_bom no)
 		(on_board yes)
 		(dnp no)
 		(fields_autoplaced yes)
 		(property "Reference" "Q1"
-			(at 128.27 35.5599 0)
+			(at 128.27 34.2899 0)
 			(effects
 				(font
@@
 			)
 		)
-		(property "Value" "S8050"
-			(at 128.27 38.0999 0)
+		(property "Value" "RE1C"
+			(at 128.27 36.8299 0)
 			(effects
 				(font
@@
 			)
 		)
-		(property "Footprint" "Resistor_SMD:R_0603_1608Metric"
-			(at 128.27 38.735 0)
-			(effects
-				(font
+		(property "Footprint" "Package_TO_SOT_SMD:SOT-416"
+			(at 128.27 39.3699 0)
+			(effects
+				(font

Commit message: pcb
Parts:
- removed R19: 0, Resistor_SMD:R_0603_1608Metric, symbol Device:R_Small
- JP2, JP6: footprint (none) -> Jumper:SolderJumper-2_P1.3mm_Open_RoundedPad1.0x1.5mm
Connections:
- net +3.3V: now also C3.1, C4.1, JP2.2 (B), U2.8 (VCC)
- net VCC_RF: now reaches R22.2
- net VCC_RF: now also L1.1
