File: Kartrack_Main_Board/LORA.kicad_sch (KiCad schematic)
At the start: 2 parts, among them J3 Conn_Coaxial, U3 Ai-Thinker-Ra-02

Commit message: BLOC schematic
Connections:
- net DIO4: now reaches U3.10 (DIO4)
- net DIO5: now reaches U3.11 (DIO5)
- net DIO0: now reaches U3.5 (DIO0)
- net DIO1: now reaches U3.6 (DIO1)
- net DIO2: now reaches U3.7 (DIO2)
- net DIO3: now reaches U3.8 (DIO3)
- no-connect marks 6 -> 0
Changed lines of the file:
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@@
 	(generator_version "9.0")
 	(paper "A4")
-	(no_connect
-		(at 138.43 99.06)
-	)
-	(no_connect
-		(at 138.43 93.98)
-	)
-	(no_connect
-		(at 138.43 96.52)
-	)
-	(no_connect
-		(at 138.43 104.14)
-	)
-	(no_connect
-		(at 138.43 101.6)
-	)
-	(no_connect
-		(at 138.43 106.68)
-	)
 	(wire
 		(pts
@@
 		)
 	)
+	(hierarchical_label "DIO2"
+		(shape input)
+		(at 138.43 99.06 0)
+		(effects
+			(font
+				(size 1.27 1.27)
+			)
+			(justify left)
+		)
+	)
 	(hierarchical_label "{slash}NSS"
 		(shape input)
@@
 			)
 			(justify right)
+		)
+	)
+	(hierarchical_label "DIO1"
+		(shape input)
+		(at 138.43 96.52 0)
+		(effects
+			(font
+				(size 1.27 1.27)
+			)
+			(justify left)
 		)
 	)
@@
 		)
 	)
+	(hierarchical_label "DIO4"
+		(shape input)
+		(at 138.43 104.14 0)
+		(effects
+			(font
+				(size 1.27 1.27)
+			)
+			(justify left)
+		)
+	)
+	(hierarchical_label "DIO5"
+		(shape input)
+		(at 138.43 106.68 0)
+		(effects
+			(font
+				(size 1.27 1.27)
+			)
+			(justify left)
+		)
+	)
+	(hierarchical_label "DIO0"
+		(shape input)
+		(at 138.43 93.98 0)
+		(effects
+			(font
+				(size 1.27 1.27)
+			)
+			(justify left)
+		)
+	)
 	(hierarchical_label "MOSI"
 		(shape input)
@@
 		)
 	)
+	(hierarchical_label "DIO3"
+		(shape input)
+		(at 138.43 101.6 0)
+		(effects
+			(font
+				(size 1.27 1.27)
+			)
+			(justify left)
+		)
+	)

Commit message: SCHEMATIC  FINISHED
Connections:
- net DIO5: no longer names the net of U3.11 (DIO5)
- no-connect marks 0 -> 1
Changed lines of the file:
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@@
 	(generator_version "9.0")
 	(paper "A4")
+	(no_connect
+		(at 138.43 106.68)
+	)
 	(wire
 		(pts
@@
 		(shape input)
 		(at 138.43 104.14 0)
-		(effects
-			(font
-				(size 1.27 1.27)
-			)
-			(justify left)
-		)
-	)
-	(hierarchical_label "DIO5"
-		(shape input)
-		(at 138.43 106.68 0)
 		(effects
 			(font
@@
 			)
 		)
+		(property "Manufacturer_Part_Number" ""
+			(at 160.02 82.55 0)
+			(effects
+				(font
+					(size 1.27 1.27)
+				)
+			)
+		)
 		(pin "1"
 		)
@@
 			)
 		)
+		(property "Manufacturer_Part_Number" ""
+			(at 128.27 99.06 0)
+			(effects
+				(font
+					(size 1.27 1.27)
+				)
+			)
+		)

Commit message: PCB early
Parts:
- J3: footprint (none) -> Connector_Coaxial:U.FL_Molex_MCRF_73412-0110_Vertical
Connections:
- net +3.3V: no longer U3.4 (~{RESET})
- new net RST: U3.4 (~{RESET})
Changed lines of the file:
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@@
-	(wire
-		(pts
-			(xy 92.71 73.66) (xy 92.71 106.68)
-		)
-		(stroke
-			(width 0)
-			(type default)
-		)
-	)
 	(wire
 		(pts
@@
 	(wire
 		(pts
-			(xy 92.71 106.68) (xy 118.11 106.68)
+			(xy 114.3 106.68) (xy 118.11 106.68)
 		)
 		(stroke
@@
 		)
 	)
+	(hierarchical_label "RST"
+		(shape input)
+		(at 114.3 106.68 180)
+		(effects
+			(font
+				(size 1.27 1.27)
+			)
+			(justify right)
+		)
+	)
 	(hierarchical_label "MOSI"
 		(shape input)
@@
 			)
 			(justify right)
-		)
-	)
-	(symbol
-		(lib_id "power:+3.3V")
-		(at 92.71 73.66 0)
-		(unit 1)
-		(exclude_from_sim no)
-		(in_bom yes)
-		(on_board yes)
-		(dnp no)
-		(fields_autoplaced yes)
-		(property "Reference" "#PWR031"
-			(at 92.71 77.47 0)
-			(effects
-				(font
-					(size 1.27 1.27)
-				)
-				(hide yes)
-			)
-		)
-		(property "Value" "+3.3V"
-			(at 92.71 68.58 0)
-			(effects
-				(font
-					(size 1.27 1.27)
-				)
-			)
-		)
-		(property "Footprint" ""
-			(at 92.71 73.66 0)
-			(effects
-				(font
-					(size 1.27 1.27)
-				)
-				(hide yes)
-			)
-		)
-		(property "Datasheet" ""
-			(at 92.71 73.66 0)
-			(effects
-				(font
-					(size 1.27 1.27)
-				)
-				(hide yes)
-			)
-		)
-		(property "Description" "Power symbol creates a global label with name \"+3.3V\""
-			(at 92.71 73.66 0)
-			(effects
-				(font
-					(size 1.27 1.27)
-				)
-				(hide yes)
-			)
-		)
-		(pin "1"
-		)
-		(instances
-			(project ""
-				(path "/7d0ecb76-dd3a-488e-b45e-ae217463e751/54cc80aa-596a-48a9-8277-047403a58fc0"
-					(reference "#PWR031")
-					(unit 1)
-				)
-			)
 		)
 	)
@@
 			)
 		)
-		(property "Footprint" ""
+		(property "Footprint" "Connector_Coaxial:U.FL_Molex_MCRF_73412-0110_Vertical"
 			(at 160.02 82.55 0)
 			(effects

Commit message: pcb
Connections:
- net GND: no longer U3.1 (ANT)
Changed lines of the file:
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@@
 		(pin "5"
-		)
-		(pin "1"
 		)
 		(pin "7"
